File: hardware/PCBs/nodemcu_board/nodemcu_board.kicad_pcb (KiCad board)
At the start: 2 copper layers, 10 parts, among them J1 USB, J2 Servo, U1 NodeMCUV3

Commit message: fix: nodemcu_board fix footprints and added rst control line
Parts:
- D1: value Cond. LED -> LED
- J1: footprint Connector_USB:USB_Micro-B_Amphenol_10103594-0001LF_Horizontal -> Connector_USB:USB_Micro-B_Molex_47346-0001
Connections:
- U1 pad 1: Net-(C1-Pad2) -> (no net)
- U1 pad 13: (no net) -> Net-(C1-Pad2)
- U1 pad 15: Net-(U1-Pad15) -> Net-(U1-Pad12)
Routing:
- net Net-(U1-Pad12): track 0.00 -> 43.3 mm
- net Net-(C1-Pad2): track 124.6 -> 94.1 mm
- net Net-(C1-Pad1): track 103.1 -> 104.2 mm
Other:
- board text added: "JLCJLCJLCJLC"
- board text added: "fish feeder board mk. 1"
