File: hardware/PCBs/nodemcu_board/nodemcu_board.sch (KiCad schematic (older format))
At the start: 6 parts, among them J1 USB, J2 Servo, U1 NodeMCUV3

Commit message: fix: nodemcu_board fix footprints and added rst control line
Parts:
- J1: footprint Connector_USB:USB_Micro-B_Amphenol_10103594-0001LF_Horizontal -> Connector_USB:USB_Micro-B_Molex_47346-0001
- U1: symbol RF_Module:NodeMCUV3 -> nodemcu_board-rescue:NodeMCUV3-RF_Module
Connections:
- net at U1.12 (RST): now also U1.15 (D0)
Changed lines of the file:
@@
 F 0 "J1" H 3757 4467 50  0000 C CNN
 F 1 "USB" H 3757 4376 50  0000 C CNN
-F 2 "Connector_USB:USB_Micro-B_Amphenol_10103594-0001LF_Horizontal" H 3850 3950 50  0001 C CNN
+F 2 "Connector_USB:USB_Micro-B_Molex_47346-0001" H 3850 3950 50  0001 C CNN
 F 3 "~" H 3850 3950 50  0001 C CNN
 	1    3700 4000
@@
 	4500 3200 5550 3200
 $Comp
-L RF_Module:NodeMCUV3 U1
+L nodemcu_board-rescue:NodeMCUV3-RF_Module U1
 U 1 1 61297303
 P 5700 4200
@@
 Wire Wire Line
 	5700 5000 6500 5000
+Wire Wire Line
+	5400 3850 5900 3850
+Wire Wire Line
+	5900 3850 5900 3800
+Wire Wire Line
+	5900 3800 6000 3800
 $EndSCHEMATC
