File: hardware/PCBs/wemos_board/wemos_board.kicad_pcb (KiCad board)
At the start: 2 copper layers, 40 x 65 mm, 10 parts, among them J1 USB, J2 Servo, U1 WeMos_D1_mini

Commit message: fix: wemos_board fix footprints and added rst control line
Parts:
- J1: footprint Connector_USB:USB_Micro-B_Amphenol_10103594-0001LF_Horizontal -> Connector_USB:USB_Micro-B_Molex_47346-0001
Connections:
- U1 pad 3: Net-(U1-Pad3) -> Net-(U1-Pad1)
Routing:
- net Net-(U1-Pad1): track 0.00 -> 12.6 mm
